Commit message: add virtual_palm

File: cpp/urdf/tocabi.urdf (robot description, URDF)
Before this commit: robot dyros_tocabi_description, 62 links, 61 joints
Links:
- added link virtual_palm
Joints:
- added joint virtual_palm_joint: type fixed, parent palm, child virtual_palm, origin rpy=0 0 1.5707963
